File: bell/bell.kicad_sch (KiCad schematic)
At the start: 106 parts, among them J4 USB_C_Receptacle_USB2.0, U1 CH32V003FxUx, U2 ME6211A33M3G-N, U3 USBLC6-2P6, U4 SN74LVC1T45DCK

Commit message: export schematic as pdf
Parts:
- D73, D74, D75, D76, D77, D78: now fitted
Changed lines of the file:
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@@
 		(in_bom yes)
 		(on_board yes)
-		(dnp yes)
+		(dnp no)
 		(property "Reference" "D76"
 			(at 212.725 97.2693 0)
@@
 		(in_bom yes)
 		(on_board yes)
-		(dnp yes)
+		(dnp no)
 		(property "Reference" "D74"
 			(at 182.245 97.2693 0)
@@
 		(in_bom yes)
 		(on_board yes)
-		(dnp yes)
+		(dnp no)
 		(property "Reference" "D73"
 			(at 167.005 97.2693 0)
@@
 		(in_bom yes)
 		(on_board yes)
-		(dnp yes)
+		(dnp no)
 		(property "Reference" "D78"
 			(at 243.205 97.2693 0)
@@
 		(in_bom yes)
 		(on_board yes)
-		(dnp yes)
+		(dnp no)
 		(property "Reference" "D75"
 			(at 197.485 97.2693 0)
@@
 		(in_bom yes)
 		(on_board yes)
-		(dnp yes)
+		(dnp no)
 		(property "Reference" "D77"
 			(at 227.965 97.2693 0)
